File: hardware/teensy2.0/parbox_t2.sch (KiCad schematic (older format))
At the start: 17 parts, among them J1 DB25_Male, J2 Debug Header, J3 I2C OLED, J4 I2C Extra, J5 ENC28J60 Module, J6 NET Select, J7 SD Card Breakout, J8 EN_EXT_INT, J9 AVR ISP, U1 Teensy2.0_(C), U2 WIZ820IO, U3 LM1117-3.3

Commit message: hw: update t2 rev 1.4
Parts:
- removed J2: Debug Header, Connector_PinHeader_2.54mm:PinHeader_1x04_P2.54mm_Vertical, symbol Connector:Conn_01x04_Female
- removed J6: NET Select, Jumper:SolderJumper-3_P1.3mm_Open_RoundedPad1.0x1.5mm_NumberLabels, symbol Connector:Conn_01x03_Male
- removed J8: EN_EXT_INT, Jumper:SolderJumper-2_P1.3mm_Bridged_RoundedPad1.0x1.5mm, symbol Connector:Conn_01x02_Male
- added J2: Debug, Connector_PinHeader_2.54mm:PinHeader_1x05_P2.54mm_Vertical, symbol Connector:Conn_01x05_Male
- added J6: ESP32 AirLift, Connector_PinHeader_2.54mm:PinHeader_1x09_P2.54mm_Vertical, symbol Connector:Conn_01x09_Male
- added R1, R2: 4k7, Resistor_SMD:R_0805_2012Metric_Pad1.15x1.40mm_HandSolder, symbol Device:R
- H1, H2, H3: footprint MountingHole:MountingHole_2.7mm_M2.5_Pad -> MountingHole:MountingHole_2.7mm_M2.5_ISO14580_Pad
- J1: footprint modules:DSUB-25_Female_EdgeMount_P2.77mm -> modules:DSUB-25_Male_EdgeMount_P2.77mm
Connections:
- net EN_INT is gone; now on net EXT_INT: J5.2 (Pin_2), U2.J1-6 (nINT)
- net SS_ENC is gone; now on net SS0: J5.7 (Pin_7)
- net SS_WIZ is gone; now on net SS0: U2.J1-5 (nSS)
- net EXT_INT: now also J2.3 (Pin_3), J6.8 (Pin_8)
- net EXT_RST: now also J6.9 (Pin_9)
- net GND: now also J2.1 (Pin_1), J6.3 (Pin_3)
- net LED: now also J2.5 (Pin_5)
- net MISO: now also J6.5 (Pin_5)
- net MOSI: now also J6.6 (Pin_6)
- net RST: now also J2.2 (Pin_2)
- net SCL: now also R1.2
- net SCLK: now also J6.4 (Pin_4)
- net SDA: now also R2.2
- net SS0: now also J6.7 (Pin_7)
- net TXD: now also J2.4 (Pin_4)
- net VCC: now also J6.1 (Pin_1), R1.1, R2.1
- no-connect marks 7 -> 8
Other:
- moved on the sheet: J1, J9
