File: hardware/pb_base/pb_base.kicad_pcb (KiCad board)
At the start: 2 copper layers, 58.4 x 80.3 mm, 19 parts, among them J1 DB25_Male, J2 MCU, J3 SPI0, J4 SPI1, J5 I2C0, J6 I2C1, J7 EXT_5V, J8 SER, U1 LevelShifter_4, U2 LevelShifter_4, U3 LevelShifter_4, U4 LevelShifter_4

Commit message: hw: updated base and pico to 0.2
Parts:
- added JP4: SolderJumper_2_Open, Connector_PinHeader_2.54mm:PinHeader_1x02_P2.54mm_Vertical, F.Cu at (80.0, 101.6)
- added JP5: SolderJumper_2_Open, Connector_PinHeader_2.54mm:PinHeader_1x02_P2.54mm_Vertical, F.Cu at (100.3, 101.6)
- JP1: footprint Jumper:SolderJumper-3_P1.3mm_Bridged2Bar12_Pad1.0x1.5mm_NumberLabels -> Connector_PinHeader_2.54mm:PinHeader_1x03_P2.54mm_Vertical
- JP2, JP3: footprint Jumper:SolderJumper-2_P1.3mm_Open_Pad1.0x1.5mm -> Connector_PinHeader_2.54mm:PinHeader_1x02_P2.54mm_Vertical
- moved JP1 8.88 mm to (89.5, 48.3), turned to -90 degrees
- moved JP3 2.55 mm to (92.7, 101.6), turned to 180 degrees
- moved JP2 2.54 mm to (87.6, 101.6)
Connections:
- J5 pad 6: /RESET -> Net-(J5-Pad6)
- J6 pad 6: /RESET -> Net-(J6-Pad6)
- U4 pad 2: /EXT1_3V3 -> /EXT1
- U4 pad 5: /EXT2_3V3 -> /EXT2
- U4 pad 6: /EXT3_3V3 -> /EXT3
Routing:
- net /EXT1: track 33.2 -> 79.9 mm
- net /EXT2: track 26.9 -> 53.1 mm
- net /EXT3: track 0.00 -> 13.9 mm
- net /+5V_PAR: track 46.3 -> 34.5 mm
- net GND: track 196.2 -> 186.7 mm
- net +3V3: track 163.3 -> 153.8 mm
- net /+5V_LVL: track 62.6 -> 57.1 mm, vias 1 -> 0
- net VCC: track 36.6 -> 42.0 mm
- net /RESET: track 72.5 -> 77.8 mm
- net /EXT3_5V: track 22.5 -> 27.0 mm
- net /SEL: track 25.6 -> 30.0 mm
- net Net-(J5-Pad6): track 0.00 -> 3.81 mm
- net Net-(J6-Pad6): track 0.00 -> 3.81 mm
- net /EXT1_5V: track 33.0 -> 30.5 mm
- net /EXT2_5V: track 30.6 -> 29.6 mm
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- added copper zone on B.Cu, net (none)
- removed copper zone on B.Cu, net GND
Other:
- board text added: "5V_MCU"
- board text added: "5V_PAR"
- board text added: "v0.2 2022 lallafa"
- board text removed: "v0.1 2022 lallafa"
