File: hardware/pb_base/pb_base.kicad_sch (KiCad schematic)
At the start: 19 parts, among them J1 DB25_Male, J2 MCU, J3 SPI0, J4 SPI1, J5 I2C0, J6 I2C1, J7 EXT_5V, J8 SER, U1 LevelShifter_4, U2 LevelShifter_4, U3 LevelShifter_4, U4 LevelShifter_4

Commit message: hw: updated base and pico to 0.2
Parts:
- added JP4, JP5: SolderJumper_2_Open, Connector_PinHeader_2.54mm:PinHeader_1x02_P2.54mm_Vertical, symbol Jumper:SolderJumper_2_Open
- JP1: footprint Jumper:SolderJumper-3_P1.3mm_Bridged2Bar12_Pad1.0x1.5mm_NumberLabels -> Connector_PinHeader_2.54mm:PinHeader_1x03_P2.54mm_Vertical
- JP2, JP3: footprint Jumper:SolderJumper-2_P1.3mm_Open_Pad1.0x1.5mm -> Connector_PinHeader_2.54mm:PinHeader_1x02_P2.54mm_Vertical
Connections:
- net EXT1_3V3 is gone; now on net EXT1: U4.2 (LV2)
- net EXT2_3V3 is gone; now on net EXT2: U4.5 (LV3)
- net EXT3_3V3 is gone; now on net EXT3: U4.6 (LV4)
- net RESET: now also JP4.2 (B), JP5.2 (B); no longer J5.6 (Pin_6), J6.6 (Pin_6)
- new net: J5.6 (Pin_6), JP4.1 (A)
- new net: J6.6 (Pin_6), JP5.1 (A)
Changed lines of the file:
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@@
   (title_block
     (title "ParBox Base Board")
-    (date "2022-02-10")
-    (rev "0.1")
+    (date "2022-03-01")
+    (rev "0.2")
   )
   (junction (at 43.18 68.58) (diameter 0) (color 0 0 0 0)
   )
   (junction (at 43.18 73.66) (diameter 0) (color 0 0 0 0)
+  )
+  (junction (at 220.98 121.92) (diameter 0) (color 0 0 0 0)
   )
   (junction (at 43.18 58.42) (diameter 0) (color 0 0 0 0)
@@
     (stroke (width 0) (type default) (color 0 0 0 0))
   )
-  (wire (pts (xy 201.93 138.43) (xy 214.63 138.43))
+  (wire (pts (xy 201.93 138.43) (xy 220.98 138.43))
     (stroke (width 0) (type default) (color 0 0 0 0))
   )
@@
     (stroke (width 0) (type default) (color 0 0 0 0))
   )
+  (wire (pts (xy 220.98 121.92) (xy 261.62 121.92))
+    (stroke (width 0) (type default) (color 0 0 0 0))
+  )
   (wire (pts (xy 114.3 154.94) (xy 114.3 151.13))
     (stroke (width 0) (type default) (color 0 0 0 0))
@@
     (stroke (width 0) (type default) (color 0 0 0 0))
   )
-  (wire (pts (xy 242.57 138.43) (xy 255.27 138.43))
+  (wire (pts (xy 242.57 138.43) (xy 261.62 138.43))
+    (stroke (width 0) (type default) (color 0 0 0 0))
+  )
+  (wire (pts (xy 220.98 138.43) (xy 220.98 132.08))
     (stroke (width 0) (type default) (color 0 0 0 0))
   )
@@
     (stroke (width 0) (type default) (color 0 0 0 0))
   )
+  (wire (pts (xy 261.62 121.92) (xy 261.62 124.46))
+    (stroke (width 0) (type default) (color 0 0 0 0))
+  )
   (wire (pts (xy 119.38 120.65) (xy 127 120.65))
     (stroke (width 0) (type default) (color 0 0 0 0))
@@
     (stroke (width 0) (type default) (color 0 0 0 0))
   )
+  (wire (pts (xy 195.58 121.92) (xy 220.98 121.92))
+    (stroke (width 0) (type default) (color 0 0 0 0))
+  )
   (wire (pts (xy 161.29 129.54) (xy 176.53 129.54))
     (stroke (width 0) (type default) (color 0 0 0 0))
@@
     (stroke (width 0) (type default) (color 0 0 0 0))
   )
+  (wire (pts (xy 261.62 132.08) (xy 261.62 138.43))
+    (stroke (width 0) (type default) (color 0 0 0 0))
+  )
   (wire (pts (xy 50.8 91.44) (xy 30.48 91.44))
     (stroke (width 0) (type default) (color 0 0 0 0))
@@
     (stroke (width 0) (type default) (color 0 0 0 0))
   )
+  (wire (pts (xy 220.98 124.46) (xy 220.98 121.92))
+    (stroke (width 0) (type default) (color 0 0 0 0))
+  )
   (wire (pts (xy 43.18 53.34) (xy 43.18 58.42))
     (stroke (width 0) (type default) (color 0 0 0 0))
@@
     (effects (font (size 1.27 1.27)) (justify left bottom))
   )
-  (label "RESET" (at 203.2 138.43 0)
-    (effects (font (size 1.27 1.27)) (justify left bottom))
-  )
   (label "SSEL1" (at 231.14 41.91 0)
     (effects (font (size 1.27 1.27)) (justify left bottom))
@@
     (effects (font (size 1.27 1.27)) (justify left bottom))
   )
+  (label "RESET" (at 195.58 121.92 0)
+    (effects (font (size 1.27 1.27)) (justify left bottom))
+  )
   (label "DATA3" (at 207.01 34.29 0)
     (effects (font (size 1.27 1.27)) (justify left bottom))
@@
     (effects (font (size 1.27 1.27)) (justify left bottom))
   )
-  (label "EXT1_3V3" (at 95.25 165.1 0)
+  (label "EXT1" (at 95.25 165.1 0)
     (effects (font (size 1.27 1.27)) (justify left bottom))
   )
@@
     (effects (font (size 1.27 1.27)) (justify left bottom))
   )
-  (label "EXT3_3V3" (at 95.25 170.18 0)
+  (label "EXT3" (at 95.25 170.18 0)
     (effects (font (size 1.27 1.27)) (justify left bottom))
   )
@@
     (effects (font (size 1.27 1.27)) (justify left bottom))
   )
-  (label "RESET" (at 243.84 138.43 0)
-    (effects (font (size 1.27 1.27)) (justify left bottom))
-  )
   (label "EXT2_5V" (at 120.65 167.64 0)
     (effects (font (size 1.27 1.27)) (justify left bottom))
@@
     (effects (font (size 1.27 1.27)) (justify left bottom))
   )
-  (label "EXT2_3V3" (at 95.25 167.64 0)
+  (label "EXT2" (at 95.25 167.64 0)
     (effects (font (size 1.27 1.27)) (justify left bottom))
   )
@@
       (effects (font (size 1.27 1.27)) (justify left) hide)
     )
-    (property "Footprint" "Jumper:SolderJumper-3_P1.3mm_Bridged2Bar12_Pad1.0x1.5mm_NumberLabels" (id 2) (at 73.66 83.82 0)
+    (property "Footprint" "Connector_PinHeader_2.54mm:PinHeader_1x03_P2.54mm_Vertical" (id 2) (at 73.66 83.82 0)
       (effects (font (size 1.27 1.27)) hide)
     )
@@
     (pin "1")
   )
+  (symbol (lib_id "Jumper:SolderJumper_2_Open") (at 261.62 128.27 90) (unit 1)
+    (in_bom yes) (on_board yes) (fields_autoplaced)
+    (property "Reference" "JP5" (id 0) (at 264.16 128.2699 90)
+      (effects (font (size 1.27 1.27)) (justify right))
+    )
+    (property "Value" "SolderJumper_2_Open" (id 1) (at 257.81 128.27 0)
+      (effects (font (size 1.27 1.27)) hide)
+    )
+    (property "Footprint" "Connector_PinHeader_2.54mm:PinHeader_1x02_P2.54mm_Vertical" (id 2) (at 261.62 128.27 0)
+      (effects (font (size 1.27 1.27)) hide)
+    )
+    (property "Datasheet" "~" (id 3) (at 261.62 128.27 0)
+      (effects (font (size 1.27 1.27)) hide)
+    )
+    (pin "1")
+    (pin "2")
+  )
   (symbol (lib_id "power:+3.3V") (at 109.22 71.12 0) (unit 1)
     (in_bom yes) (on_board yes) (fields_autoplaced)
@@
       (effects (font (size 1.27 1.27)) hide)
     )
-    (property "Footprint" "Jumper:SolderJumper-2_P1.3mm_Open_Pad1.0x1.5mm" (id 2) (at 208.28 128.27 0)
+    (property "Footprint" "Connector_PinHeader_2.54mm:PinHeader_1x02_P2.54mm_Vertical" (id 2) (at 208.28 128.27 0)
       (effects (font (size 1.27 1.27)) hide)
     )
@@
       (effects (font (size 1.27 1.27)) hide)
     )
-    (property "Footprint" "Jumper:SolderJumper-2_P1.3mm_Open_Pad1.0x1.5mm" (id 2) (at 248.92 128.27 0)
+    (property "Footprint" "Connector_PinHeader_2.54mm:PinHeader_1x02_P2.54mm_Vertical" (id 2) (at 248.92 128.27 0)
       (effects (font (size 1.27 1.27)) hide)
     )
@@
     )
     (pin "1")
+  )
+  (symbol (lib_id "Jumper:SolderJumper_2_Open") (at 220.98 128.27 90) (unit 1)
+    (in_bom yes) (on_board yes) (fields_autoplaced)
+    (property "Reference" "JP4" (id 0) (at 223.52 128.2699 90)
+      (effects (font (size 1.27 1.27)) (justify right))
+    )
+    (property "Value" "SolderJumper_2_Open" (id 1) (at 217.17 128.27 0)
+      (effects (font (size 1.27 1.27)) hide)
+    )
+    (property "Footprint" "Connector_PinHeader_2.54mm:PinHeader_1x02_P2.54mm_Vertical" (id 2) (at 220.98 128.27 0)
+      (effects (font (size 1.27 1.27)) hide)
+    )
+    (property "Datasheet" "~" (id 3) (at 220.98 128.27 0)
+      (effects (font (size 1.27 1.27)) hide)
+    )
+    (pin "1")
+    (pin "2")
   )
   (symbol (lib_id "power:GND") (at 166.37 104.14 0) (unit 1)
@@
     )
     (path "/083fe946-e982-48e1-ad71-6cbbb6edfd5a"
-      (reference "JP1") (unit 1) (value "SolderJumper_3_Bridged12") (footprint "Jumper:SolderJumper-3_P1.3mm_Bridged2Bar12_Pad1.0x1.5mm_NumberLabels")
+      (reference "JP1") (unit 1) (value "SolderJumper_3_Bridged12") (footprint "Connector_PinHeader_2.54mm:PinHeader_1x03_P2.54mm_Vertical")
     )
     (path "/5c8eb51b-7ac2-4865-a61e-387859536da3"
-      (reference "JP2") (unit 1) (value "SolderJumper_2_Open") (footprint "Jumper:SolderJumper-2_P1.3mm_Open_Pad1.0x1.5mm")
+      (reference "JP2") (unit 1) (value "SolderJumper_2_Open") (footprint "Connector_PinHeader_2.54mm:PinHeader_1x02_P2.54mm_Vertical")
     )
     (path "/9146468e-5a9d-4395-8259-86ab44524974"
-      (reference "JP3") (unit 1) (value "SolderJumper_2_Open") (footprint "Jumper:SolderJumper-2_P1.3mm_Open_Pad1.0x1.5mm")
+      (reference "JP3") (unit 1) (value "SolderJumper_2_Open") (footprint "Connector_PinHeader_2.54mm:PinHeader_1x02_P2.54mm_Vertical")
+    )
+    (path "/b8475d55-603f-4665-a6ee-f583099b1be1"
+      (reference "JP4") (unit 1) (value "SolderJumper_2_Open") (footprint "Connector_PinHeader_2.54mm:PinHeader_1x02_P2.54mm_Vertical")
+    )
+    (path "/3c77bfe7-86c5-40d5-bb7b-ccef38595622"
+      (reference "JP5") (unit 1) (value "SolderJumper_2_Open") (footprint "Connector_PinHeader_2.54mm:PinHeader_1x02_P2.54mm_Vertical")
     )
     (path "/faaff343-1d6b-4119-87dc-80081ab16200"
