File: hardware/pb_cpu_pipico/pb_cpu_pipico.kicad_pcb (KiCad board)
At the start: 2 copper layers, 55.9 x 48.3 mm, 6 parts, among them J1 MCU, SW1 Reset, U1 Pico

Commit message: hw: updated base and pico to 0.2
Connections:
- U1 pad 1: /TX -> /TXD
- U1 pad 2: /RX -> /RXD
- U1 pad 35: GND -> +3V3
- U1 pad 37: +3V3 -> unconnected-(U1-Pad37)
Routing:
- net VCC: track 61.2 -> 87.9 mm
- net /TXD: track 0.00 -> 14.8 mm
- net /RXD: track 0.00 -> 14.8 mm
- net /EXT1: track 62.9 -> 49.3 mm
- net /SSEL0: track 51.7 -> 41.5 mm
- net /MOSI: track 50.0 -> 40.8 mm
- net /SCK: track 55.5 -> 47.1 mm
- net /SSEL1: track 36.0 -> 43.0 mm, vias 0 -> 1
- net GND: track 131.0 -> 136.8 mm
- net /STROBE: track 33.6 -> 38.6 mm
- net /SEL: track 18.3 -> 15.8 mm
- net /INT1: track 39.2 -> 37.2 mm, vias 1 -> 0
- net /RESET: track 54.6 -> 52.7 mm
- net +3V3: track 49.3 -> 51.1 mm
Other:
- board text added: "v0.2 2022 lallafa"
- board text removed: "v0.1 2022 lallafa"
