File: hardware/pb_cpu_pipico/pb_cpu_pipico.kicad_sch (KiCad schematic)
At the start: 6 parts, among them J1 MCU, SW1 Reset, U1 Pico

Commit message: hw: updated base and pico to 0.2
Connections:
- net RX is gone; now on net RXD: U1.2 (GPIO1)
- net TX is gone; now on net TXD: U1.1 (GPIO0)
- net +3V3: now also U1.35 (ADC_VREF); no longer U1.37 (3V3_EN)
- net GND: no longer U1.35 (ADC_VREF)
- no-connect marks 5 -> 6
Changed lines of the file:
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@@
   (title_block
     (title "AmiParBox CPU Board Pi Pico")
-    (date "2022-02-11")
-    (rev "0.1")
+    (date "2022-03-01")
+    (rev "0.2")
   )
   (junction (at 201.93 69.85) (diameter 0) (color 0 0 0 0)
   )
-  (junction (at 201.93 52.07) (diameter 0) (color 0 0 0 0)
-  )
-  (junction (at 186.69 49.53) (diameter 0) (color 0 0 0 0)
+  (junction (at 208.28 49.53) (diameter 0) (color 0 0 0 0)
   )
   (junction (at 129.54 82.55) (diameter 0) (color 0 0 0 0)
@@
   (no_connect (at 78.74 73.66))
   (no_connect (at 78.74 76.2))
+  (no_connect (at 181.61 46.99))
   (no_connect (at 161.29 92.71))
   (no_connect (at 163.83 92.71))
@@
     (stroke (width 0) (type default) (color 0 0 0 0))
   )
-  (wire (pts (xy 201.93 52.07) (xy 201.93 57.15))
+  (wire (pts (xy 201.93 44.45) (xy 201.93 57.15))
     (stroke (width 0) (type default) (color 0 0 0 0))
   )
@@
     (stroke (width 0) (type default) (color 0 0 0 0))
   )
-  (wire (pts (xy 201.93 44.45) (xy 201.93 52.07))
-    (stroke (width 0) (type default) (color 0 0 0 0))
-  )
-  (wire (pts (xy 186.69 49.53) (xy 208.28 49.53))
-    (stroke (width 0) (type default) (color 0 0 0 0))
-  )
   (wire (pts (xy 181.61 39.37) (xy 184.15 39.37))
     (stroke (width 0) (type default) (color 0 0 0 0))
@@
     (stroke (width 0) (type default) (color 0 0 0 0))
   )
-  (wire (pts (xy 181.61 49.53) (xy 186.69 49.53))
+  (wire (pts (xy 181.61 49.53) (xy 208.28 49.53))
     (stroke (width 0) (type default) (color 0 0 0 0))
   )
@@
     (stroke (width 0) (type default) (color 0 0 0 0))
   )
+  (wire (pts (xy 181.61 52.07) (xy 208.28 52.07))
+    (stroke (width 0) (type default) (color 0 0 0 0))
+  )
   (wire (pts (xy 135.89 87.63) (xy 146.05 87.63))
     (stroke (width 0) (type default) (color 0 0 0 0))
@@
     (stroke (width 0) (type default) (color 0 0 0 0))
   )
-  (wire (pts (xy 181.61 46.99) (xy 186.69 46.99))
-    (stroke (width 0) (type default) (color 0 0 0 0))
-  )
   (wire (pts (xy 135.89 74.93) (xy 146.05 74.93))
     (stroke (width 0) (type default) (color 0 0 0 0))
   )
-  (wire (pts (xy 181.61 52.07) (xy 201.93 52.07))
-    (stroke (width 0) (type default) (color 0 0 0 0))
-  )
   (wire (pts (xy 44.45 78.74) (xy 44.45 81.28))
     (stroke (width 0) (type default) (color 0 0 0 0))
@@
     (stroke (width 0) (type default) (color 0 0 0 0))
   )
+  (wire (pts (xy 208.28 52.07) (xy 208.28 49.53))
+    (stroke (width 0) (type default) (color 0 0 0 0))
+  )
   (wire (pts (xy 129.54 82.55) (xy 146.05 82.55))
     (stroke (width 0) (type default) (color 0 0 0 0))
@@
     (stroke (width 0) (type default) (color 0 0 0 0))
   )
-  (wire (pts (xy 186.69 46.99) (xy 186.69 49.53))
-    (stroke (width 0) (type default) (color 0 0 0 0))
-  )
   (wire (pts (xy 181.61 64.77) (xy 208.28 64.77))
     (stroke (width 0) (type default) (color 0 0 0 0))
@@
     (effects (font (size 1.27 1.27)) (justify left bottom))
   )
-  (label "TX" (at 135.89 39.37 0)
+  (label "TXD" (at 135.89 39.37 0)
     (effects (font (size 1.27 1.27)) (justify left bottom))
   )
@@
     (effects (font (size 1.27 1.27)) (justify left bottom))
   )
-  (label "RX" (at 135.89 41.91 0)
-    (effects (font (size 1.27 1.27)) (justify left bottom))
-  )
+  (label "RXD" (at 135.89 41.91 0)
+    (effects (font (size 1.27 1.27)) (justify left bottom))
+  )
